File: 51-02.kicad_pcb (KiCad board)
At the start: 2 copper layers, 50 x 72 mm, 0 parts

Commit message: first net generarted
Parts:
- added C1: 100nF, 01_vtech-snom-footprints:C_0805_vtech-snom, F.Cu at (72.0, 84.8)
- added C2: 1uF, 01_vtech-snom-footprints:C_0805_vtech-snom, F.Cu at (88.6, 54.7)
- added C3: 1uF, 01_vtech-snom-footprints:C_0805_vtech-snom, F.Cu at (84.1, 59.3)
- added FID1: Fiducial, 01_vtech-snom-footprints:1-DA_Fiducial_1.5mm_Mask3mm, F.Cu at (63.0, 128.8)
- added FID2: Fiducial, 01_vtech-snom-footprints:1-DA_Fiducial_1.5mm_Mask3mm, F.Cu at (84.4, 55.6)
- added J1: 1_DA_Conn_02x14_Counter_Clockwise, 01_vtech-snom-footprints:1-DA_PinHeader_2x14_P2.00mm_Vertical, F.Cu at (148.8, 70.0)
- added J2: Conn_01x28_I, 01_vtech-snom-footprints:1_DA_PinHeader_I_1x28_P2.54mm_Vertical, F.Cu at (63.0, 55.7)
- added J3: Conn_01x28_II, 01_vtech-snom-footprints:1_DA_PinHeader_II_1x28_P2.54mm_Vertical, F.Cu at (67.7, 55.7)
- added J4: 1_DA_Conn_02x14_Counter_Clockwise, 01_vtech-snom-footprints:1-DA_PinHeader_2x14_P2.00mm_Vertical, F.Cu at (110.7, 69.9)
- added R1: 4K7, 01_vtech-snom-footprints:R_0805_vtech-snom, F.Cu at (88.0, 59.3)
- added R2: 4K7, 01_vtech-snom-footprints:R_0805_vtech-snom, F.Cu at (92.0, 57.5)
- added R3: 4K7, 01_vtech-snom-footprints:R_0805_vtech-snom, F.Cu at (95.9, 54.7)
- added R4: 4K7, 01_vtech-snom-footprints:R_0805_vtech-snom, F.Cu at (99.9, 54.7)

Commit message: first complete release
Parts:
- moved FID2 90.1 mm to (150.0, 117.3)
- moved FID1 87.7 mm to (107.5, 53.2)
- moved J3 69.2 mm to (136.7, 51.3)
- moved C2 59.5 mm to (142.0, 80.9), turned to 270 degrees
- moved J2 58.8 mm to (121.7, 51.3)
- moved C1 44.3 mm to (114.6, 72.6), turned to 270 degrees
- moved C3 31.5 mm to (112.6, 72.6), turned to 270 degrees
- moved R2 25.0 mm to (116.9, 59.0), turned to 270 degrees
- moved R1 22.9 mm to (110.9, 59.0), turned to 270 degrees
- moved R3 19.5 mm to (114.9, 59.0), turned to 270 degrees
- moved R4 13.7 mm to (112.9, 59.0), turned to 270 degrees
- moved J4 4.39 mm to (107.2, 72.6)
- moved J1 2.68 mm to (149.2, 72.6)
Connections:
- C1 pad 1: Net-(C1-Pad1) -> VDD
- C2 pad 1: Net-(C1-Pad1) -> VDD
- C3 pad 1: Net-(C1-Pad1) -> VDD
- J1 pad 10: (no net) -> Net-(J1-Pad10)
- J1 pad 11: (no net) -> Net-(J1-Pad11)
- J1 pad 12: (no net) -> Net-(J1-Pad12)
- J1 pad 13: (no net) -> Net-(J1-Pad13)
- J1 pad 14: (no net) -> Net-(J1-Pad14)
- J1 pad 15: (no net) -> Net-(J1-Pad15)
- J1 pad 16: (no net) -> Net-(J1-Pad16)
- J1 pad 17: (no net) -> Net-(J1-Pad17)
- J1 pad 18: (no net) -> Net-(J1-Pad18)
- J1 pad 19: (no net) -> Net-(J1-Pad19)
- J1 pad 20: (no net) -> Net-(J1-Pad20)
- J1 pad 21: (no net) -> Net-(J1-Pad21)
- J1 pad 22: (no net) -> Net-(J1-Pad22)
- J1 pad 23: (no net) -> Net-(J1-Pad23)
- J1 pad 24: (no net) -> Net-(J1-Pad24)
- J1 pad 25: (no net) -> Net-(J1-Pad25)
- J1 pad 4: (no net) -> Net-(J1-Pad4)
- J1 pad 5: (no net) -> Net-(J1-Pad5)
- J1 pad 6: (no net) -> Net-(J1-Pad6)
- J1 pad 8: (no net) -> Net-(J1-Pad8)
- J1 pad 9: (no net) -> Net-(J1-Pad9)
- J2 pad 1: (no net) -> Net-(J2-Pad1)
- J2 pad 11: (no net) -> Net-(J2-Pad11)
- J2 pad 12: (no net) -> VDD
- J2 pad 2: (no net) -> Net-(J2-Pad2)
- J2 pad 20: (no net) -> Net-(J2-Pad20)
- J2 pad 21: (no net) -> Net-(J2-Pad21)
- J2 pad 22: (no net) -> Net-(J2-Pad22)
- J2 pad 23: (no net) -> Net-(J2-Pad23)
- J2 pad 24: (no net) -> Net-(J2-Pad24)
- J2 pad 25: (no net) -> Net-(J2-Pad25)
- J2 pad 26: (no net) -> Net-(J2-Pad26)
- J2 pad 27: (no net) -> Net-(J2-Pad27)
- J2 pad 28: (no net) -> Net-(J2-Pad28)
- J2 pad 3: (no net) -> Net-(J2-Pad3)
- J3 pad 29: (no net) -> Net-(J3-Pad29)
- J3 pad 30: (no net) -> Net-(J3-Pad30)
- J3 pad 31: (no net) -> Net-(J3-Pad31)
- J3 pad 32: (no net) -> Net-(J3-Pad32)
- J3 pad 42: Net-(J3-Pad42) -> VDD
- J3 pad 45: Net-(J3-Pad42) -> VDD
- J3 pad 46: (no net) -> Net-(J3-Pad46)
- J3 pad 47: Net-(J3-Pad42) -> VDD
- J3 pad 52: /DQS -> /IO7
- J4 pad 14: /DQS -> /IO7
- J4 pad 2: (no net) -> Net-(J4-Pad2)
- J4 pad 26: (no net) -> Net-(J4-Pad26)
- J4 pad 27: (no net) -> Net-(J4-Pad27)
- J4 pad 28: (no net) -> VDD
Routing:
- net /IO7: track 0.00 -> 70.9 mm
- net /IO6: track 0.00 -> 66.0 mm
- net /RB3: track 0.00 -> 62.1 mm
- net /IO15: track 0.00 -> 62.0 mm, vias 0 -> 1
- net /IO5: track 0.00 -> 61.4 mm
- net /IO14: track 0.00 -> 57.7 mm, vias 0 -> 3
- net /IO4: track 0.00 -> 57.3 mm
- net /IO3: track 0.00 -> 56.5 mm, vias 0 -> 2
- net VDD: track 0.00 -> 56.2 mm
- net /IO13: track 0.00 -> 55.9 mm, vias 0 -> 1
- net GND: track 0.00 -> 53.5 mm, vias 0 -> 10
- net /RB1: track 0.00 -> 50.3 mm, vias 0 -> 1
- net /IO12: track 0.00 -> 49.8 mm
- net /IO11: track 0.00 -> 49.2 mm, vias 0 -> 2
- net /IO8: track 0.00 -> 47.1 mm, vias 0 -> 1
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- added copper zone on B.Cu, net GND
Other:
- net class Net Class 1 added: clearance 0.2, trace_width 0.5, via_dia 0.8, via_drill 0.4

Commit message: silk+3d
Parts:
- added G***: LOGO, 51-pretty:RohS-loggo-2.9mm_x_2.9mm, F.Cu at (139.3, 112.1)
- added G***: LOGO, 51-pretty:ESD-logo-3.1mm_x_2.6mm, F.Cu at (143.7, 109.3)
- added G***: LOGO, 51-pretty:E-trash-logo-3.2mm_x_4.6mm, F.Cu at (147.5, 108.1)
- added G***: LOGO, 51-pretty:CE-logo-2.9mm_x_2_9mm, F.Cu at (143.6, 106.9)
- added REF**: 51_OSHW-Logo2_7.3x6mm, 01_vtech-snom-footprints:51_OSHW-Logo2_7.3x6mm, F.Cu at (148.1, 60.8)
- J2: value Conn_01x28_I -> Conn_01x24_I; footprint 01_vtech-snom-footprints:1_DA_PinHeader_I_1x28_P2.54mm_Vertical -> 01_vtech-snom-footprints:1-DA_PinHeader_I_1x24_P2.54mm_Vertical
- J3: value Conn_01x28_II -> Conn_01x24_II; footprint 01_vtech-snom-footprints:1_DA_PinHeader_II_1x28_P2.54mm_Vertical -> 01_vtech-snom-footprints:1-DA_PinHeader_II_1x24_P2.54mm_Vertical
- moved FID2 8.92 mm to (151.7, 108.5)
Routing:
- net /RB3: track 62.1 -> 56.8 mm
Other:
- board size 50 x 72 mm -> 50 x 61.4 mm
- board text added: "48-pin-adapter 360-clip set + FlashcatUSB XPORT"
- board text added: "51-02-01-01"
- board text added: "Copyright©2021 1-DA"
