File: 51-02.sch (KiCad schematic (older format))
At the start: 4 parts

Commit message: sch first release
Parts:
- removed J? (x2): 1_DA_Conn_02x14_Odd_Even, 01_vtech-snom-footprints:1_DA_PinHeader_2x14_P1.27mm_Vertical, symbol 01_vtech-snom:1_DA_Conn_02x14_Odd_Even
- removed J? (x2): Conn_01x28, 01_vtech-snom-footprints:1_DA_PinHeader_1x28_P2.54mm_Vertical, symbol 01_vtech-snom:Conn_01x28
- added C1: 100nF, 01_vtech-snom-footprints:C_0805_vtech-snom, symbol 01_vtech-snom:C0805
- added C2, C3: 1uF, 01_vtech-snom-footprints:C_0805_vtech-snom, symbol 01_vtech-snom:C0805
- added FID1, FID2: Fiducial, 01_vtech-snom-footprints:1-DA_Fiducial_1.5mm_Mask3mm, symbol 01_vtech-snom:Fiducial
- added J1, J4: 1_DA_Conn_02x14_Counter_Clockwise, 01_vtech-snom-footprints:1_DA_PinHeader_2x14_clock-wise_P1.27mm_Vertical, symbol 01_vtech-snom:1_DA_Conn_02x14_Counter_Clockwise
- added J2: Conn_01x28_I, 01_vtech-snom-footprints:1_DA_PinHeader_I_1x28_P2.54mm_Vertical, symbol 01_vtech-snom:Conn_01x28_I
- added J3: Conn_01x28_II, 01_vtech-snom-footprints:1_DA_PinHeader_II_1x28_P2.54mm_Vertical, symbol 01_vtech-snom:Conn_01x28_II
- added R1, R2, R3, R4: 4K7, 01_vtech-snom-footprints:R_0805_vtech-snom, symbol 01_vtech-snom:R0805_5%
Connections:
- new net: J3.42 (Pin_42), J3.45 (Pin_45), J3.47 (Pin_47)
- new net: C1.1, C2.1, C3.1
- new net A0_CE1: J1.1 (Pin_1), J2.10 (Pin_10)
- new net A1_CE2: J1.2 (Pin_2), J2.14 (Pin_14)
- new net A2_CE3: J1.3 (Pin_3), J2.15 (Pin_15)
- new net ALE: J2.17 (Pin_17), J4.4 (Pin_4)
- new net CE0: J2.9 (Pin_9), J4.24 (Pin_24)
- new net CLE: J2.16 (Pin_16), J4.3 (Pin_3)
- new net DQS: J3.43 (Pin_43), J3.52 (Pin_52), J4.14 (Pin_14), J4.23 (Pin_23)
- new net GND: C1.2, C2.2, C3.2, J2.13 (Pin_13), J3.33 (Pin_33), J3.44 (Pin_44), J3.56 (Pin_56), J4.1 (Pin_1), R1.1, R2.1, R3.1, R4.1
- new net IO0: J3.37 (Pin_37), J4.7 (Pin_7)
- new net IO1: J3.38 (Pin_38), J4.8 (Pin_8)
- new net IO10: J3.36 (Pin_36), J4.20 (Pin_20)
- new net IO11: J3.41 (Pin_41), J4.19 (Pin_19)
- new net IO12: J3.48 (Pin_48), J4.18 (Pin_18)
- new net IO13: J3.53 (Pin_53), J4.17 (Pin_17)
- new net IO14: J3.54 (Pin_54), J4.16 (Pin_16)
- new net IO15: J3.55 (Pin_55), J4.15 (Pin_15)
- new net IO2: J3.39 (Pin_39), J4.9 (Pin_9)
- new net IO3: J3.40 (Pin_40), J4.10 (Pin_10)
- new net IO4: J3.49 (Pin_49), J4.11 (Pin_11)
- new net IO5: J3.50 (Pin_50), J4.12 (Pin_12)
- new net IO6: J3.51 (Pin_51), J4.13 (Pin_13)
- new net IO8: J3.34 (Pin_34), J4.22 (Pin_22)
- new net IO9: J3.35 (Pin_35), J4.21 (Pin_21)
- new net RB: J2.7 (Pin_7), J4.6 (Pin_6), R1.2
- new net RB1: J1.28 (Pin_28), J2.6 (Pin_6), R4.2
- new net RB2: J1.27 (Pin_27), J2.5 (Pin_5), R3.2
- new net RB3: J1.26 (Pin_26), J2.4 (Pin_4), R2.2
- new net RE: J2.8 (Pin_8), J4.5 (Pin_5)
- new net WE: J2.18 (Pin_18), J4.25 (Pin_25)
- new net WP: J1.7 (Pin_7), J2.19 (Pin_19)
- no-connect marks 0 -> 42
Other:
- note added: "1"
- note added: "24"
- note added: "25"
- note added: "26"
- note added: "27"
- note added: "28"
- note added: "29"
- note added: "30"
- note added: "31\n"
- note added: "32"
- note added: "33"
- note added: "34"
- note added: "35"
- note added: "36"
- note added: "37"
- note added: "39"
- note added: "40"
- note added: "41"
- note added: "42"
- note added: "43"
- note added: "44"
- note added: "45"
- note added: "46"
- note added: "47"
- note added: "48"
- note added: "48-pin TSOP1\nStandard Type"

Commit message: 2x14 2mm raster
Parts:
- J1, J4: footprint 01_vtech-snom-footprints:1_DA_PinHeader_2x14_clock-wise_P1.27mm_Vertical -> 01_vtech-snom-footprints:1-DA_PinHeader_2x14_P2.00mm_Vertical
Changed lines of the file:
@@
 F 0 "J4" H 9050 4425 50  0000 C CNN
 F 1 "1_DA_Conn_02x14_Counter_Clockwise" H 9050 4426 50  0001 C CNN
-F 2 "01_vtech-snom-footprints:1_DA_PinHeader_2x14_clock-wise_P1.27mm_Vertical" H 9000 3700 50  0001 C CNN
+F 2 "01_vtech-snom-footprints:1-DA_PinHeader_2x14_P2.00mm_Vertical" H 9000 3700 50  0001 C CNN
 F 3 "~" H 9000 3700 50  0001 C CNN
 	1    9000 3700
@@
 F 0 "J1" H 2550 4325 50  0000 C CNN
 F 1 "1_DA_Conn_02x14_Counter_Clockwise" H 2550 4326 50  0001 C CNN
-F 2 "01_vtech-snom-footprints:1_DA_PinHeader_2x14_clock-wise_P1.27mm_Vertical" H 2500 3600 50  0001 C CNN
+F 2 "01_vtech-snom-footprints:1-DA_PinHeader_2x14_P2.00mm_Vertical" H 2500 3600 50  0001 C CNN
 F 3 "~" H 2500 3600 50  0001 C CNN
 	1    2500 3600
@@
 L power:GND #PWR04
 U 1 1 606C206E
-P 4800 3650
-F 0 "#PWR04" H 4800 3400 50  0001 C CNN
-F 1 "GND" H 4805 3477 50  0001 C CNN
-F 2 "" H 4800 3650 50  0001 C CNN
-F 3 "" H 4800 3650 50  0001 C CNN
-	1    4800 3650
+P 3800 3650
+F 0 "#PWR04" H 3800 3400 50  0001 C CNN
+F 1 "GND" H 3805 3477 50  0001 C CNN
+F 2 "" H 3800 3650 50  0001 C CNN
+F 3 "" H 3800 3650 50  0001 C CNN
+	1    3800 3650
 	0    1    1    0
 $EndComp
-Wire Wire Line
-	4800 3650 5300 3650
 Text Notes 6500 3700 0    50   ~ 0
 36
@@
 Wire Wire Line
 	8250 1750 8250 1950
+Wire Wire Line
+	3800 3650 5300 3650
 $EndSCHEMATC

Commit message: first complete release
Connections:
- net DQS: no longer J3.52 (Pin_52), J4.14 (Pin_14)
- net VDD: now reaches J2.12 (Pin_12)
- net VDD: now also C1.1, C2.1, C3.1, J3.42 (Pin_42), J3.45 (Pin_45), J3.47 (Pin_47), J4.28 (Pin_28)
- new net IO7: J3.52 (Pin_52), J4.14 (Pin_14)
Changed lines of the file:
@@
-	1    0    0    -1
-$EndComp
-$Comp
-L 01_vtech-snom:3V3_SYS #PWR07
-U 1 1 606C90CD
-P 6600 1150
-F 0 "#PWR07" H 6600 1150 50  0001 C CNN
-F 1 "3V3_SYS" H 6600 1373 50  0000 C CNN
-F 2 "" H 6600 1150 50  0001 C CNN
-F 3 "" H 6600 1150 50  0001 C CNN
-	1    6600 1150
 	1    0    0    -1
 $EndComp
@@
 Wire Wire Line
 	7200 1350 7800 1350
-$Comp
-L 01_vtech-snom:3V3_SYS #PWR01
-U 1 1 606CAF19
-P 3700 3500
-F 0 "#PWR01" H 3700 3500 50  0001 C CNN
-F 1 "3V3_SYS" H 3700 3723 50  0000 C CNN
-F 2 "" H 3700 3500 50  0001 C CNN
-F 3 "" H 3700 3500 50  0001 C CNN
-	1    3700 3500
-	1    0    0    -1
-$EndComp
 Text Notes 6500 3900 0    50   ~ 0
 34
@@
 Wire Wire Line
 	7500 3350 7500 3300
-$Comp
-L 01_vtech-snom:3V3_SYS #PWR09
-U 1 1 606CDFFF
-P 7500 3250
-F 0 "#PWR09" H 7500 3250 50  0001 C CNN
-F 1 "3V3_SYS" H 7500 3473 50  0000 C CNN
-F 2 "" H 7500 3250 50  0001 C CNN
-F 3 "" H 7500 3250 50  0001 C CNN
-	1    7500 3250
-	1    0    0    -1
-$EndComp
 Connection ~ 7500 3550
 Wire Wire Line
@@
 Wire Wire Line
 	6850 3750 7850 3750
-Text Label 8600 4400 0    50   ~ 0
-DQS
 Text Label 7850 3750 0    50   ~ 0
 DQS
-$Comp
-L 01_vtech-snom:3V3_SYS #PWR012
-U 1 1 607472D8
-P 9500 2950
-F 0 "#PWR012" H 9500 2950 50  0001 C CNN
-F 1 "3V3_SYS" H 9500 3173 50  0000 C CNN
-F 2 "" H 9500 2950 50  0001 C CNN
-F 3 "" H 9500 2950 50  0001 C CNN
-	1    9500 2950
-	1    0    0    -1
-$EndComp
 Wire Wire Line
 	9300 3100 9500 3100
-Wire Wire Line
-	9500 3100 9500 3000
 NoConn ~ 9300 3200
 NoConn ~ 9300 3300
@@
 Connection ~ 8250 1750
 Wire Wire Line
+	8250 1750 8250 1950
+Wire Wire Line
+	3800 3650 5300 3650
+Wire Wire Line
+	9500 3000 9500 3100
+Wire Wire Line
 	6600 1200 6600 1350
-Wire Wire Line
-	8250 1750 8250 1950
-Wire Wire Line
-	3800 3650 5300 3650
+$Comp
+L power:VDD #PWR0101
+U 1 1 60743265
+P 6600 1200
+F 0 "#PWR0101" H 6600 1050 50  0001 C CNN
+F 1 "VDD" H 6615 1373 50  0000 C CNN
+F 2 "" H 6600 1200 50  0001 C CNN
+F 3 "" H 6600 1200 50  0001 C CNN
+	1    6600 1200
+	1    0    0    -1
+$EndComp
+$Comp
+L power:VDD #PWR0102
+U 1 1 60744C09
+P 9500 3000
+F 0 "#PWR0102" H 9500 2850 50  0001 C CNN
+F 1 "VDD" H 9515 3173 50  0000 C CNN
+F 2 "" H 9500 3000 50  0001 C CNN
+F 3 "" H 9500 3000 50  0001 C CNN
+	1    9500 3000
+	1    0    0    -1
+$EndComp
+$Comp
+L power:VDD #PWR0103
+U 1 1 607457ED
+P 7500 3300
+F 0 "#PWR0103" H 7500 3150 50  0001 C CNN
+F 1 "VDD" H 7515 3473 50  0000 C CNN
+F 2 "" H 7500 3300 50  0001 C CNN
+F 3 "" H 7500 3300 50  0001 C CNN
+	1    7500 3300
+	1    0    0    -1
+$EndComp
+$Comp
+L power:VDD #PWR0104
+U 1 1 607461D0
+P 3700 3500
+F 0 "#PWR0104" H 3700 3350 50  0001 C CNN
+F 1 "VDD" H 3715 3673 50  0000 C CNN
+F 2 "" H 3700 3500 50  0001 C CNN
+F 3 "" H 3700 3500 50  0001 C CNN
+	1    3700 3500
+	1    0    0    -1
+$EndComp
+Wire Wire Line
+	3700 3550 3700 3500
+$Comp
+L power:PWR_FLAG #FLG0101
+U 1 1 6074AC6A
+P 7200 1150
+F 0 "#FLG0101" H 7200 1225 50  0001 C CNN
+F 1 "PWR_FLAG" H 7200 1323 50  0000 C CNN
+F 2 "" H 7200 1150 50  0001 C CNN
+F 3 "~" H 7200 1150 50  0001 C CNN
+	1    7200 1150
+	1    0    0    -1
+$EndComp
+Wire Wire Line
+	7200 1350 7200 1150
 $EndSCHEMATC

Commit message: silk+3d
Parts:
- removed J2: Conn_01x28_I, 01_vtech-snom-footprints:1_DA_PinHeader_I_1x28_P2.54mm_Vertical, symbol 01_vtech-snom:Conn_01x28_I
- removed J3: Conn_01x28_II, 01_vtech-snom-footprints:1_DA_PinHeader_II_1x28_P2.54mm_Vertical, symbol 01_vtech-snom:Conn_01x28_II
- added J2: Conn_01x24_I, 01_vtech-snom-footprints:1-DA_PinHeader_I_1x24_P2.54mm_Vertical, symbol 01_vtech-snom:Conn_01x24_I
- added J3: Conn_01x24_II, 01_vtech-snom-footprints:1-DA_PinHeader_II_1x24_P2.54mm_Vertical, symbol 01_vtech-snom:Conn_01x24_II
Connections:
- net A0_CE1: now also J2.10 (Pin_10)
- net A1_CE2: now also J2.14 (Pin_14)
- net A2_CE3: now also J2.15 (Pin_15)
- net ALE: now also J2.17 (Pin_17)
- net CE0: now also J2.9 (Pin_9)
- net CLE: now also J2.16 (Pin_16)
- net DQS: now also J3.43 (Pin_43)
- net GND: now also J2.13 (Pin_13), J3.33 (Pin_33), J3.44 (Pin_44), J3.56 (Pin_56)
- net IO0: now also J3.37 (Pin_37)
- net IO1: now also J3.38 (Pin_38)
- net IO10: now also J3.36 (Pin_36)
- net IO11: now also J3.41 (Pin_41)
- net IO12: now also J3.48 (Pin_48)
- net IO13: now also J3.53 (Pin_53)
- net IO14: now also J3.54 (Pin_54)
- net IO15: now also J3.55 (Pin_55)
- net IO2: now also J3.39 (Pin_39)
- net IO3: now also J3.40 (Pin_40)
- net IO4: now also J3.49 (Pin_49)
- net IO5: now also J3.50 (Pin_50)
- net IO6: now also J3.51 (Pin_51)
- net IO7: now also J3.52 (Pin_52)
- net IO8: now also J3.34 (Pin_34)
- net IO9: now also J3.35 (Pin_35)
- net RB: now also J2.7 (Pin_7)
- net RB1: now also J2.6 (Pin_6)
- net RB2: now also J2.5 (Pin_5)
- net RB3: now also J2.4 (Pin_4)
- net RE: now also J2.8 (Pin_8)
- net VDD: now also J2.12 (Pin_12), J3.42 (Pin_42), J3.45 (Pin_45), J3.47 (Pin_47)
- net WE: now also J2.18 (Pin_18)
- net WP: now also J2.19 (Pin_19)
- no-connect marks 42 -> 34
Changed lines of the file:
@@
 encoding utf-8
 Sheet 1 1
-Title "56-pin-adapter for the 360-clip set and FlashcatUSB XPORT"
+Title "48-pin-adapter for the 360-clip set and FlashcatUSB XPORT"
 Date ""
 Rev "01"
@@
 Comment4 ""
 $EndDescr
-$Comp
-L 01_vtech-snom:Conn_01x28_I J2
-U 1 1 606AFD56
-P 5500 3750
-F 0 "J2" H 5500 5200 50  0000 L CNN
-F 1 "Conn_01x28_I" H 5500 2250 50  0001 C CNN
-F 2 "01_vtech-snom-footprints:1_DA_PinHeader_I_1x28_P2.54mm_Vertical" H 5500 3750 50  0001 C CNN
-F 3 "~" H 5500 3750 50  0001 C CNN
-	1    5500 3750
-	1    0    0    -1
-$EndComp
-$Comp
-L 01_vtech-snom:Conn_01x28_II J3
-U 1 1 606B0E27
-P 6650 3750
-F 0 "J3" H 6568 5175 50  0000 C CNN
-F 1 "Conn_01x28_II" H 6650 2250 50  0001 C CNN
-F 2 "01_vtech-snom-footprints:1_DA_PinHeader_II_1x28_P2.54mm_Vertical" H 6650 3750 50  0001 C CNN
-F 3 "~" H 6650 3750 50  0001 C CNN
-	1    6650 3750
-	-1   0    0    -1
-$EndComp
 Text Notes 5600 2500 0    50   ~ 0
 1
@@
 Text Label 9500 4100 0    50   ~ 0
 IO12
-NoConn ~ 5300 4850
-NoConn ~ 5300 4950
-NoConn ~ 5300 5050
-NoConn ~ 5300 5150
-NoConn ~ 6850 5150
-NoConn ~ 6850 5050
-NoConn ~ 6850 4950
-NoConn ~ 6850 4850
 NoConn ~ 8800 3200
 Wire Wire Line
@@
 Wire Wire Line
 	7200 1350 7200 1150
+$Comp
+L 01_vtech-snom:Conn_01x24_I J2
+U 1 1 6073CFA6
+P 5500 3750
+F 0 "J2" H 5450 5150 50  0000 L CNN
+F 1 "Conn_01x24_I" H 5500 2250 50  0001 C CNN
+F 2 "01_vtech-snom-footprints:1-DA_PinHeader_I_1x24_P2.54mm_Vertical" H 5500 3750 50  0001 C CNN
+F 3 "~" H 5500 3750 50  0001 C CNN
+	1    5500 3750
+	1    0    0    -1
+$EndComp
+$Comp
+L 01_vtech-snom:Conn_01x24_II J3
+U 1 1 60742D7D
+P 6650 3750
+F 0 "J3" H 6650 5150 50  0000 C CNN
+F 1 "Conn_01x24_II" H 6650 2250 50  0001 C CNN
+F 2 "01_vtech-snom-footprints:1-DA_PinHeader_II_1x24_P2.54mm_Vertical" H 6650 3750 50  0001 C CNN
+F 3 "~" H 6650 3750 50  0001 C CNN
+	1    6650 3750
+	-1   0    0    -1
+$EndComp
 $EndSCHEMATC
